File: 386_memory_board_simm.kicad_sch (KiCad schematic)
At the start: 73 parts, among them J1 Bus_386_Memory, U10 74LS174, U11 74LS174, U12 74LS174, U13 74LS174, U14 74LS158, U15 74LS158, U16 74LS158, U17 7410, U18 SPARE, U19 SPARE, U37 7410, U38 7400, U39 7400, U40 7410, U43 7402, U44 7410, U45 74LS04, U5 74LS174, U6 74LS174, U7 74LS158, U8 74LS158, U9 74LS158

Commit message: fixed footprint of delay lines
Parts:
- U20, U22: footprint Package_SO:SO-16_5.3x10.2mm_P1.27mm -> Package_SO:SOIC-16W_7.5x12.8mm_P1.27mm
Changed lines of the file:
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@@
 			)
 		)
-		(property "Footprint" "Package_SO:SO-16_5.3x10.2mm_P1.27mm"
+		(property "Footprint" "Package_SO:SOIC-16W_7.5x12.8mm_P1.27mm"
 			(at 229.87 295.91 0)
 			(effects
@@
 			)
 		)
-		(property "Footprint" "Package_SO:SO-16_5.3x10.2mm_P1.27mm"
+		(property "Footprint" "Package_SO:SOIC-16W_7.5x12.8mm_P1.27mm"
 			(at 66.04 297.18 0)
 			(effects

Commit message: added bracket mounting holes
Parts:
- U17, U37, U40, U44: value 7410 -> 74F10
- U38, U39: value 7400 -> 74F00
- U43: value 7402 -> 74F02
Changed lines of the file:
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@@
 			)
 		)
-		(property "Value" "7402"
+		(property "Value" "74F02"
 			(at 499.11 403.86 0)
 			(effects
@@
 			)
 		)
-		(property "Value" "7400"
+		(property "Value" "74F00"
 			(at 105.41 394.97 90)
 			(effects
@@
 			)
 		)
-		(property "Value" "7410"
+		(property "Value" "74F10"
 			(at 180.34 450.8814 0)
 			(effects
@@
 			)
 		)
-		(property "Value" "7400"
+		(property "Value" "74F00"
 			(at 269.24 338.074 0)
 			(effects
@@
 			)
 		)
-		(property "Value" "7410"
+		(property "Value" "74F10"
 			(at 608.33 105.4414 0)
 			(effects
@@
 			)
 		)
-		(property "Value" "7410"
+		(property "Value" "74F10"
 			(at 280.67 295.9414 0)
 			(effects
@@
 			)
 		)
-		(property "Value" "7410"
+		(property "Value" "74F10"
 			(at 115.57 250.2214 0)
 			(effects
@@
 			)
 		)
-		(property "Value" "7410"
+		(property "Value" "74F10"
 			(at 280.67 318.8014 0)
 			(effects
@@
 			)
 		)
-		(property "Value" "7400"
+		(property "Value" "74F00"
 			(at 269.24 352.552 0)
 			(effects
@@
 			)
 		)
-		(property "Value" "7400"
+		(property "Value" "74F00"
 			(at 105.4017 381 0)
 			(effects
@@
 			)
 		)
-		(property "Value" "7410"
+		(property "Value" "74F10"
 			(at 151.13 450.8814 0)
 			(effects
@@
 			)
 		)
-		(property "Value" "7402"
+		(property "Value" "74F02"
 			(at 497.84 375.92 0)
 			(effects
@@
 			)
 		)
-		(property "Value" "7400"
+		(property "Value" "74F00"
 			(at 269.24 366.268 0)
 			(effects
@@
 			)
 		)
-		(property "Value" "7410"
+		(property "Value" "74F10"
 			(at 115.57 274.3514 0)
 			(effects
@@
 			)
 		)
-		(property "Value" "7402"
+		(property "Value" "74F02"
 			(at 631.19 111.76 90)
 			(effects
@@
 			)
 		)
-		(property "Value" "7410"
+		(property "Value" "74F10"
 			(at 115.57 297.2114 0)
 			(effects
@@
 			)
 		)
-		(property "Value" "7400"
+		(property "Value" "74F00"
 			(at 269.24 393.7 90)
 			(effects
@@
 			)
 		)
-		(property "Value" "7410"
+		(property "Value" "74F10"
 			(at 115.57 320.0714 0)
 			(effects
@@
 			)
 		)
-		(property "Value" "7402"
+		(property "Value" "74F02"
 			(at 631.19 97.79 0)
 			(effects
@@
 			)
 		)
-		(property "Value" "7400"
+		(property "Value" "74F00"
 			(at 269.24 380.492 0)
 			(effects
@@
 			)
 		)
-		(property "Value" "7410"
+		(property "Value" "74F10"
 			(at 280.67 250.2214 0)
 			(effects
@@
 			)
 		)
-		(property "Value" "7400"
+		(property "Value" "74F00"
 			(at 105.4017 339.09 0)
 			(effects
@@
 			)
 		)
-		(property "Value" "7402"
+		(property "Value" "74F02"
 			(at 631.19 55.88 0)
 			(effects
@@
 			)
 		)
-		(property "Value" "7400"
+		(property "Value" "74F00"
 			(at 105.4017 367.03 0)
 			(effects
@@
 			)
 		)
-		(property "Value" "7410"
+		(property "Value" "74F10"
 			(at 280.67 273.0814 0)
 			(effects
@@
 			)
 		)
-		(property "Value" "7400"
+		(property "Value" "74F00"
 			(at 105.4017 353.06 0)
 			(effects

Commit message: PCB Revision 2 -implements 8MB operation -fixed the missing slot cutout on rev.1 -overhauls the slot connector based on i440bx's discoveries and design -add information to modify rev.1 Boards to 8MB
Parts:
- added H1, H2: MountingHole, MountingHole:MountingHole_3.2mm_M3_DIN965_Pad, symbol Mechanical:MountingHole
- added J2, J3: Conn_01x02_Pin, Connector_PinHeader_2.54mm:PinHeader_1x02_P2.54mm_Vertical, symbol Connector:Conn_01x02_Pin
- added RP7A1, RP7B1: 100, symbol Device:R
- added RP9A1, RP9B1: 10k, symbol Device:R_Pack08
- added U139, U25, U26: PAL16L8, symbol Logic_Programmable:PAL16L8
- added U141: PAL20L8, symbol Logic_Programmable:PAL20L8
- added U160: 74LS74, symbol 74xx:74LS74
- added U46: 74LS590, symbol 74xx:74LS590
- added U67: 74LS158, symbol 74xx:74LS158
- added U73, U74: 74LS373, symbol 74xx:74LS373
Connections:
- net A5A: now also U67.4 (Za)
- net A6A: now also U67.7 (Zb)
- net A7A: now also U67.9 (Zd)
- net A8A: now also U67.12 (Zc)
- net PIN100: now also U73.2 (O0), U73.5 (O1); no longer J1.100, U43.8
- net PIN101: now also U74.2 (O0), U74.5 (O1); no longer J1.101, U43.6
- net CPUA21: now reaches J1.85 (CPUA21)
- net CPUA21: now also J2.2 (Pin_2)
- net CPUA22: now reaches J1.95 (CPUA22)
- net CPUA22: now also J3.2 (Pin_2)
- net A9B: now reaches U10.4 (D1)
- net A9B: now also U13.4 (D1), J3.1 (Pin_1)
- net A9A: now reaches U9.5 (I0b)
- net A9A: now also U16.5 (I0b), J2.1 (Pin_1)
- net PIN103 renamed RMSEL0
- net PIN104 renamed RMSEL1
- net PIN105 renamed MEMREF
- net ~{PIN105} renamed ~{MEMREF}
- new net: RP7A1.1, U67.15 (E)
- new net: U160.11 (C), U46.9 (~{RCO})
- new net: U160.12 (D), U160.8 (~{Q})
- new net: U160.9 (Q), U67.14 (I0c)
- new net: RP7B1.1, U73.1 (OE), U74.1 (OE)
- new net: U25.1 (I1), U26.1 (I1)
- new net: U25.11 (I10), U26.11 (I10)
- new net: U26.18 (IO2), U73.11 (LE)
- new net: U25.2 (I2), U26.2 (I2)
- new net: U141.7 (I7), U25.4 (I4), U26.4 (I4)
- new net: U141.4 (I4), U25.5 (I5), U26.5 (I5)
- new net: U25.6 (I6), U26.6 (I6)
- new net: U25.7 (I7), U26.7 (I7)
- new net: U25.8 (I8), U26.8 (I8)
- new net: U141.20 (I020), U73.4 (D1), U74.4 (D1)
- new net: U141.21 (IO21), U73.3 (D0), U74.3 (D0)
- new net: RP9A1.8 (R8.1), U141.3 (I3)
- new net: U139.12 (IO8), U141.5 (I5), U67.1 (S)
- new net: U141.6 (I6), U25.9 (I9)
- new net: RP9A1.10 (R7.2), RP9A1.11 (R6.2), RP9A1.12 (R5.2), RP9A1.13 (R4.2), RP9A1.14 (R3.2), RP9A1.15 (R2.2), RP9A1.16 (R1.2), RP9A1.9 (R8.2), RP9B1.1 (R1.1), RP9B1.16 (R1.2), RP9B1.2 (R2.1), RP9B1.3 (R3.1), RP9B1.4 (R4.1), RP9B1.5 (R5.1), RP9B1.6 (R6.1), RP9B1.7 (R7.1), RP9B1.8 (R8.1)
- new net: U25.18 (IO2), U74.11 (LE)
- new net 386dx A11: U67.13 (I1c)
- new net E28: RP9A1.5 (R5.1), U141.23 (I23)
- new net E32: RP9A1.6 (R6.1), U141.1 (I1)
- new net E35: RP9A1.7 (R7.1), U141.2 (I2)
- new net GND: RP7A1.2, RP7B1.2
- new net SLEB0: J1.100 (SLEB0), U43.8
- new net SLEB1: J1.101 (SLEB1), U43.6
- no-connect marks 30 -> 31
Other:
- note added: "2/8M Selection open: 2M closed: 8M"
- note added: "J19"
- note added: "J20"
- note added: "not shared across slots!"
- note added: "on board stuff"
- moved on the sheet: C32, C33, U18, U19, U43B, U43C
